Commit message: define camera frame and extrinsics

File: ros2_ws/src/xle_description/urdf/xlerobot.urdf (robot description, URDF)
Before this commit: robot xlerobot, 45 links, 44 joints
Links:
- removed link head_camera_depth_frame
- removed link head_camera_rgb_frame
Joints:
- removed joint fixed_head_camera_depth_frame
- removed joint fixed_head_camera_rgb_frame
